Commit message: arm

File: turtlebot9_description/urdf/sensors/hokuyo.urdf.xacro (robot description, xacro)
@@ -24,5 +24,5 @@
  </link>
  <joint name="hokuyo_joint" type="fixed">
-   <origin xyz="0.132 0.0 0.13" rpy="3.14 0 0"/>
+   <origin xyz="0.131 0.0 0.142" rpy="3.14 0 0"/>
    <parent link="${parent}"/>
    <child link="laser_joint"/>

File: turtlebot9_description/urdf/sensors/kinect.urdf.xacro (robot description, xacro)
@@ -34,5 +34,6 @@
     </link>
   <joint name="camera_joint" type="fixed">
-    <origin xyz="-0.031 ${-cam_py} -0.016" rpy="0 0 0"/>
+  <!--  <origin xyz="-0.031 ${-cam_py} -0.016" rpy="0 0 0"/> -->
+    <origin xyz="0.1814 ${-cam_py} 0.032" rpy="0 0 0"/>
     <parent link="camera_rgb_frame"/>
     <child link="camera_link"/>

File: turtlebot9_description/urdf/stacks/hexagons.urdf.xacro (robot description, xacro)
@@ -45,5 +45,5 @@
     <link name="pole_middle_${number}_link">
       <visual>
-        <origin xyz="0 0 0" rpy="0 ${M_PI} 0"/>
+        <origin xyz="0 0 0" rpy="${M_PI} ${M_PI} 0"/>
         <geometry>
           <mesh filename="package://turtlebot_description/meshes/stacks/hexagons/pole_middle.dae"/>
@@ -138,5 +138,5 @@
       <origin xyz="0.02364 0.0 0.1307" rpy="0 0 0"/>
 -->
-      <origin xyz="0.02364 0.0 0.1507" rpy="0 0 0"/>
+      <origin xyz="0.02364 0.0 0.1807" rpy="0 0 0"/>
       <parent link="${parent}"/>
       <child link="plate_bottom_link"/>
@@ -163,8 +163,13 @@
       </inertial>
     </link>
-    <stack_middle_pole parent="${parent}" number="0" x_loc= "0.0381" y_loc= "0.1505" z_loc="0.1640"/>
-    <stack_middle_pole parent="${parent}" number="1" x_loc= "0.0381" y_loc="-0.1505" z_loc="0.1640"/>
-    <stack_middle_pole parent="${parent}" number="2" x_loc="-0.0381" y_loc= "0.1505" z_loc="0.1640"/>
-    <stack_middle_pole parent="${parent}" number="3" x_loc="-0.0381" y_loc="-0.1505" z_loc="0.1640"/>
+    <stack_middle_pole parent="${parent}" number="0" x_loc= "0.120" y_loc= "0.082" z_loc="0.1480"/>
+    <stack_middle_pole parent="${parent}" number="1" x_loc= "0.055" y_loc= "0.120" z_loc="0.1480"/>
+    <stack_middle_pole parent="${parent}" number="2" x_loc="-0.055" y_loc= "0.120" z_loc="0.1480"/>
+    <stack_middle_pole parent="${parent}" number="3" x_loc="0.120" y_loc= "-0.082" z_loc="0.1480"/>
+    <stack_middle_pole parent="${parent}" number="4" x_loc="0.055" y_loc="-0.120" z_loc="0.1480"/>
+    <stack_middle_pole parent="${parent}" number="5" x_loc="-0.055" y_loc="-0.120" z_loc="0.1480"/>
+    <stack_middle_pole parent="${parent}" number="6" x_loc="0.11" y_loc="0.098" z_loc="	0.202"/>
+    <stack_middle_pole parent="${parent}" number="7" x_loc="0.11" y_loc="-0.098" z_loc="0.202"/>
+<!--
     <joint name="plate_middle_joint" type="fixed">
       <origin xyz="-0.01364 0.0 0.1874" rpy="0 0 0"/>
@@ -193,12 +198,13 @@
       </inertial>
     </link>
-    <stack_top_pole parent="${parent}" number="0" x_loc= "0.0381" y_loc= "0.1505" z_loc="0.2920"/>
-    <stack_top_pole parent="${parent}" number="1" x_loc= "0.0381" y_loc="-0.1505" z_loc="0.2920"/>
-    <stack_top_pole parent="${parent}" number="2" x_loc="-0.0381" y_loc= "0.1505" z_loc="0.2920"/>
-    <stack_top_pole parent="${parent}" number="3" x_loc="-0.0381" y_loc="-0.1505" z_loc="0.2920"/>
-    <stack_3d_sensor_pole parent="${parent}" number="0" x_loc="-0.1024" y_loc= "0.098" z_loc="0.2372"/>
-    <stack_3d_sensor_pole parent="${parent}" number="1" x_loc="-0.1024" y_loc="-0.098" z_loc="0.2372"/>
+-->
+    <stack_top_pole parent="${parent}" number="0" x_loc= "0.0381" y_loc= "0.1505" z_loc="0.2840"/>
+    <stack_top_pole parent="${parent}" number="1" x_loc= "0.0381" y_loc="-0.1505" z_loc="0.2840"/>
+    <stack_top_pole parent="${parent}" number="2" x_loc="-0.0381" y_loc= "0.1505" z_loc="0.2840"/>
+    <stack_top_pole parent="${parent}" number="3" x_loc="-0.0381" y_loc="-0.1505" z_loc="0.2840"/>
+    <stack_3d_sensor_pole parent="${parent}" number="0" x_loc="0.11" y_loc= "0.098" z_loc="0.2792"/>
+    <stack_3d_sensor_pole parent="${parent}" number="1" x_loc="0.11" y_loc="-0.098" z_loc="0.2792"/>
     <joint name="plate_top_joint" type="fixed">
-      <origin xyz="-0.01364 0.0  0.3966" rpy="0 0 0"/>
+      <origin xyz="-0.01364 0.0  0.3886" rpy="0 0 0"/>
       <parent link="${parent}"/>
       <child link="plate_top_link"/>

File: turtlebot9_description/urdf/turtlebot9_library.urdf.xacro (robot description, xacro)
@@ -17,3 +17,4 @@
   <xacro:include filename="$(find turtlebot9_description)/urdf/sensors/asus_xtion_pro.urdf.xacro"/>
   <xacro:include filename="$(find turtlebot9_description)/urdf/sensors/hokuyo.urdf.xacro"/>
-</robot>
+<!--  <xacro:include filename="$(find turtlebot9_description)/urdf/arm/arm.urdf.xacro"/>  -->
+	</robot>
